File: SteeringWheel/SteeringWheel.kicad_pcb (KiCad board)
At the start: 2 copper layers, 4 parts, among them J1 Conn_01x02_Male, U1 RC1602A, U2 MCP23008-xP

Commit message: Layout
Parts:
- removed A2: Arduino_Nano_v2.x, Module:Arduino_Nano
- removed U2: MCP23008-xP, Package_DIP:DIP-18_W7.62mm
- added J2: Conn_01x10, TerminalBlock_Phoenix:TerminalBlock_Phoenix_MKDS-1,5-10-5.08_1x10_P5.08mm_Horizontal, F.Cu at (111.7, 97.0)
- added J3: Conn_01x16_Female, Connector_PinSocket_2.54mm:PinSocket_1x16_P2.54mm_Vertical, F.Cu at (147.5, 36.8)
- added J4: Conn_01x10_Female, TerminalBlock_Phoenix:TerminalBlock_Phoenix_MKDS-1,5-10-5.08_1x10_P5.08mm_Horizontal, F.Cu at (174.3, 84.5)
- added R1: R, Resistor_THT:R_Axial_DIN0204_L3.6mm_D1.6mm_P7.62mm_Horizontal, F.Cu at (111.9, 84.4)
- J1: footprint TerminalBlock_Phoenix:TerminalBlock_Phoenix_MKDS-1,5-2_1x02_P5.00mm_Horizontal -> TerminalBlock_Phoenix:TerminalBlock_Phoenix_MKDS-1,5-2-5.08_1x02_P5.08mm_Horizontal
- U1: value RC1602A -> ATmega8A-PU; footprint Display:RC1602A -> Package_DIP:DIP-28_W7.62mm
- moved J1 52.3 mm to (98.3, 51.0), turned to 270 degrees
- moved U1 43.4 mm to (146.2, 50.3), turned to 270 degrees
Connections:
- net Net-(J1-Pad2) renamed GND
- J1 pad 1: Net-(J1-Pad1) -> +5V
Routing:
- net Net-(J2-Pad2): track 0.00 -> 82.0 mm
- net Net-(J2-Pad3): track 0.00 -> 74.9 mm
- net Net-(J2-Pad4): track 0.00 -> 67.7 mm
- net +5V: track 0.00 -> 66.4 mm
- net Net-(J2-Pad6): track 0.00 -> 56.2 mm
- net Net-(J2-Pad10): track 0.00 -> 22.0 mm
- net Net-(R1-Pad2): track 0.00 -> 19.5 mm
- net Net-(J3-Pad5): track 0.00 -> 13.9 mm
- net Net-(J3-Pad6): track 0.00 -> 13.9 mm
- net Net-(J3-Pad4): track 0.00 -> 13.9 mm
- net Net-(J3-Pad3): track 0.00 -> 13.9 mm
- net Net-(J2-Pad1): track 0.00 -> 12.6 mm

Commit message: update
Parts:
- J2, J4: footprint TerminalBlock_Phoenix:TerminalBlock_Phoenix_MKDS-1,5-10-5.08_1x10_P5.08mm_Horizontal -> TerminalBlock_Phoenix:TerminalBlock_Phoenix_MPT-0,5-10-2.54_1x10_P2.54mm_Horizontal
- moved J1 71.7 mm to (168.8, 37.4)
- moved J2 24.5 mm to (113.1, 72.5)
- moved R1 20.6 mm to (112.0, 63.8)
- moved J4 10.2 mm to (168.5, 76.1)
- moved U1 7.76 mm to (145.1, 42.6)
Routing:
- net Net-(J2-Pad2): track 82.0 -> 0.00 mm
- net Net-(J2-Pad3): track 74.9 -> 0.00 mm
- net Net-(J2-Pad4): track 67.7 -> 0.00 mm
- net +5V: track 66.4 -> 0.00 mm
- net Net-(J2-Pad6): track 56.2 -> 0.00 mm
- net Net-(J2-Pad10): track 22.0 -> 0.00 mm
- net Net-(R1-Pad2): track 19.5 -> 0.00 mm
- net Net-(J3-Pad5): track 13.9 -> 0.00 mm
- net Net-(J3-Pad6): track 13.9 -> 0.00 mm
- net Net-(J3-Pad4): track 13.9 -> 0.00 mm
- net Net-(J3-Pad3): track 13.9 -> 0.00 mm
- net Net-(J2-Pad1): track 12.6 -> 0.00 mm
